Commit message: chore: add gazebo xacro tutorial

File: ros_ws/src/example_urdf_robot/urdf/diff_drive.urdf.xacro (robot description, xacro)
@@ -19,5 +19,5 @@
 <xacro:property name="wheel_length" value="0.06" />
 <xacro:property name="wheel_radius" value="0.10" />
-<xacro:property name="wheel_mass" value="1.20" />
+<xacro:property name="wheel_mass" value="1.2" />
 <xacro:property name="lidar_mass" value="0.12" />
 <xacro:property name="lidar_width" value="0.10" />
@@ -104,5 +104,23 @@
 <xacro:wheel name="wheel_right" length="${wheel_length}" radius="${wheel_radius}" mass="${wheel_mass}" reflect="-1"/>
 <!-- Castor Link -->
-<link name="castor_link">
+<link name="front_castor_link">
+    <visual>
+        <geometry>
+            <sphere radius="${castor_radius}"/>
+        </geometry>
+        <material name="uom_grey"/>
+    </visual>
+    <collision>
+        <geometry>
+            <sphere radius="${castor_radius}"/>
+        </geometry>
+    </collision>
+    <xacro:property name="I_castor" value="${(2/5)*castor_mass*castor_radius**2}"/>
+    <inertial>
+        <mass value="${castor_mass}"/>
+        <inertia ixx="${I_castor}" ixy="0.0" ixz="0.0" iyy="${I_castor}" iyz="0.0" izz="${I_castor}"/>
+    </inertial>
+</link>
+<link name="back_castor_link">
     <visual>
         <geometry>
@@ -140,8 +158,13 @@
     <axis xyz="0 0 1"/>
 </joint>
-<joint name="base_castor_joint" type="fixed">
+<joint name="base_front_castor_joint" type="fixed">
     <parent link="base_link"/>
-    <child link="castor_link"/>
+    <child link="front_castor_link"/>
     <origin xyz="0.3 0 ${-0.5*base_link_z + base_link_origin_z}"/>
+</joint>
+<joint name="base_back_castor_joint" type="fixed">
+    <parent link="base_link"/>
+    <child link="back_castor_link"/>
+    <origin xyz="${-base_link_origin_x} 0 ${-0.5*base_link_z + base_link_origin_z}"/>
 </joint>
 <joint name="footprint_base_joint" type="fixed">

File: ros_ws/src/example_urdf_robot/urdf/example_gazebo.xacro (robot description, xacro)
@@ -3,12 +3,16 @@
  <!-- GAZEBO PLUGINS -->
   <!-- List all movable joints -->
+  <!-- https://gazebosim.org/api/gazebo/6/classignition_1_1gazebo_1_1systems_1_1JointStatePublisher.html -->
   <gazebo>
       <plugin filename="ignition-gazebo-joint-state-publisher-system" name="ignition::gazebo::systems::JointStatePublisher">
-        <update_rate>50</update_rate>
+        <update_rate>100</update_rate>
         <joint_name>base_wheel_left_joint</joint_name>
         <joint_name>base_wheel_right_joint</joint_name>
+        <!-- <topic>/world/<world_name>/model/<model_name>/joint_state</topic> THIS IS DEFAULT -->
+        <topic>/model/diff_drive_example/joint_state</topic> <!-- remove world leading prefixes -->
       </plugin>
   </gazebo>
-  <!-- Differential Drive - https://gazebosim.org/api/gazebo/6/classignition_1_1gazebo_1_1systems_1_1DiffDrive.html -->
+  <!-- Differential Drive -->
+  <!-- https://gazebosim.org/api/gazebo/6/classignition_1_1gazebo_1_1systems_1_1DiffDrive.html -->
   <gazebo>
     <plugin filename="ignition-gazebo-diff-drive-system" name="ignition::gazebo::systems::DiffDrive">
@@ -30,4 +34,5 @@
     </plugin>
   </gazebo>
+  <!-- SENSORS -->
   <gazebo reference="lidar_link">
     <sensor type="gpu_lidar" name="generic_lidar_sensor">
@@ -35,9 +40,9 @@
       <frame_id>lidar_link</frame_id>
       <ignition_frame_id>lidar_link</ignition_frame_id>
-      <update_rate>10.0</update_rate>
+      <update_rate>15.0</update_rate>
       <ray>
         <scan>
           <horizontal>
-            <samples>512</samples>
+            <samples>270</samples>
             <resolution>1</resolution>
             <min_angle>-${pi*0.75}</min_angle>
@@ -47,15 +52,15 @@
         <range>
           <min>0.10</min>
-          <max>10.0</max>
-          <resolution>0.03</resolution>
+          <max>8.0</max>
+          <resolution>0.06</resolution>
         </range>
         <noise>
           <type>gaussian</type>
           <mean>0.0</mean>
-          <stddev>0.001</stddev>
+          <stddev>0.02</stddev>
         </noise>
       </ray>
       <always_on>1</always_on>
-      <visualize>false</visualize>
+      <visualize>true</visualize>
     </sensor>
   </gazebo>
@@ -65,9 +70,9 @@
     </plugin>
   </gazebo>
-  <gazebo reference="imu_link">
+  <gazebo reference="base_link">
     <sensor name="imu_sensor" type="imu">
       <topic>/model/diff_drive_example/imu</topic>
-      <frame_id>imu_link</frame_id>
-      <ignition_frame_id>imu_link</ignition_frame_id>
+      <frame_id>base_link</frame_id>
+      <ignition_frame_id>base_link</ignition_frame_id>
       <plugin filename="libignition-gazebo-imu-system.so" name="ignition::gazebo::systems::Imu">
         <initial_orientation_as_reference>false</initial_orientation_as_reference>
@@ -131,10 +136,15 @@
       </imu>
     </sensor>
+  </gazebo>
   <!-- FRICTION AND PHYSICS -->
-  <!-- <gazebo reference="castor_link">
-    <mu1 value="0.001"/>
-    <mu2 value="0.001"/>
-  </gazebo> -->
-  <!-- <gazebo reference="wheel_right">
+  <gazebo reference="back_castor_link">
+    <mu1 value="0.00001"/>
+    <mu2 value="0.00001"/>
+  </gazebo>
+  <gazebo reference="front_castor_link">
+    <mu1 value="0.00001"/>
+    <mu2 value="0.00001"/>
+  </gazebo>
+  <gazebo reference="wheel_right">
     <mu1 value="1.0"/>
     <mu2 value="1.0"/>
@@ -143,5 +153,4 @@
     <mu1 value="1.0"/>
     <mu2 value="1.0"/>
-  </gazebo> -->
   </gazebo>
 </robot>
